File: OmniAnt/MotorController_MCF8329A.kicad_sch (KiCad schematic)
At the start: 22 parts, among them Q1 NTMFS4C324NT1G, Q2 NTMFS4C324NT1G, Q3 NTMFS4C324NT1G, Q4 NTMFS4C324NT1G, Q5 NTMFS4C324NT1G, Q6 NTMFS4C324NT1G, U3 MCF8329A1IREER

Commit message: Mostly organizing
Parts:
- removed C10, C13, C4, C6, C8, C9: 1uF, symbol Device:C
- removed C11: 0.1uF, symbol Device:C
- removed C12: C, symbol Device:C
- removed C5, C7: 10uF, symbol Device:C
- removed Q1, Q2, Q3, Q4, Q5, Q6: NTMFS4C324NT1G, NVMFS5C442NLWFAFT1G, symbol SamacSys_Parts:NTMFS4C324NT1G
- removed R2, R3: 10k, Resistor_SMD:R_0805_2012Metric, symbol Device:R
- removed R4, R5: 5.1k, Resistor_SMD:R_0805_2012Metric, symbol Device:R
- removed U3: MCF8329A1IREER, REE0036A-IPC_A, symbol MCF8329A:MCF8329A1IREER
- added C1, C11, C14, C19, C2, C20: 1uF, PCM_JLCPCB:C_0603, symbol PCM_JLCPCB-Capacitors:0603,1uF
- added C21: 100nF, PCM_JLCPCB:C_0603, symbol PCM_JLCPCB-Capacitors:0603,100nF
- added C4: 470pF, PCM_JLCPCB:C_0603, symbol PCM_JLCPCB-Capacitors:0603,470pF
- added C6, C8: 10uF, PCM_JLCPCB:C_0805, symbol PCM_JLCPCB-Capacitors:0805,10uF,(2)
- added Q10, Q11, Q12, Q8, Q9: NTMFS4C324NT1G, NVMFS5C442NLWFAFT1G, symbol NTMFS4C324NT1G:NTMFS4C324NT1G
- added Q7: NTMFS4C324NT1G, Footprints:NVMFS5C442NLWFAFT1G, symbol NTMFS4C324NT1G:NTMFS4C324NT1G
- added R10, R9: 5.1kΩ, PCM_JLCPCB:R_0402, symbol PCM_JLCPCB-Resistors:0402,5.1kΩ
- added R3, R4: 10kΩ, PCM_JLCPCB:R_0402, symbol PCM_JLCPCB-Resistors:0402,10kΩ
- added U3: MCF8329A1IREER, Footprints:REE0036A-MFG, symbol CustomParts:MCF8329A1IREER
Connections:
- net +3.3V: now also R10.1, R9.1
- net 3.3V: now also C11.1, U3.2 (VREG), U3.27 (SPEED_WAKE)
- net Batt: now also C21.1, C6.1, Q11.5 (D_1), Q11.6 (D_2), Q11.7 (D_3), Q11.8 (D_4), Q11.9 (D_5), Q7.5 (D_1), Q7.6 (D_2), Q7.7 (D_3), Q7.8 (D_4), Q7.9 (D_5), Q9.5 (D_1), Q9.6 (D_2), Q9.7 (D_3), Q9.8 (D_4), Q9.9 (D_5), U3.5 (PVDD)
- net DACOut: now also U3.33 (DACOUT_SOx_SPEED_ANA)
- net GND: now also C1.2, C11.2, C2.2, C21.2, C6.2, C8.2, R3.1, R4.1, U3.1 (DGND), U3.23 (SN), U3.25 (AGND), U3.37 (Thermal_pad), U3.4 (GND)
- net LSS: now also Q10.1 (S_1), Q10.2 (S_2), Q10.3 (S_3), Q12.1 (S_1), Q12.2 (S_2), Q12.3 (S_3), Q8.1 (S_1), Q8.2 (S_2), Q8.3 (S_3), U3.21 (LSS), U3.22 (SP)
- net SCL: now also U3.30 (SCL)
- net SDA: now also U3.29 (SDA)
- new net: Q10.4 (G), U3.16 (GLB)
- new net: Q10.5 (D_1), Q10.6 (D_2), Q10.7 (D_3), Q10.8 (D_4), Q10.9 (D_5), Q9.1 (S_1), Q9.2 (S_2), Q9.3 (S_3)
- new net: R10.2, U3.35 (FAULT_N)
- new net: Q12.4 (G), U3.20 (GLC)
- new net: Q11.1 (S_1), Q11.2 (S_2), Q11.3 (S_3), Q12.5 (D_1), Q12.6 (D_2), Q12.7 (D_3), Q12.8 (D_4), Q12.9 (D_5)
- new net: C14.2, Q7.1 (S_1), Q7.2 (S_2), Q7.3 (S_3), Q8.5 (D_1), Q8.6 (D_2), Q8.7 (D_3), Q8.8 (D_4), Q8.9 (D_5), U3.10 (SHA)
- new net: Q7.4 (G), U3.11 (GHA)
- new net: C14.1, U3.9 (BSTA)
- new net: R4.2, U3.34 (BRAKE)
- new net: Q11.4 (G), U3.19 (GHC)
- new net: Q8.4 (G), U3.12 (GLA)
- new net: C8.1, U3.8 (GVDD)
- new net: C2.1, U3.36 (DVDD)
- new net: C4.1, U3.7 (CPH)
- new net: C4.2, U3.6 (CPL)
- new net: C1.1, U3.26 (AVDD)
- new net: Q9.4 (G), U3.15 (GHB)
- new net: R9.2, U3.28 (FG)
- new net: C19.1, U3.13 (BSTB)
- new net: C19.2, U3.14 (SHB)
- new net: C20.1, U3.17 (BSTC)
- new net: C20.2, U3.18 (SHC)
- new net: R3.2, U3.31 (DIR)

Commit message: Good progress on the power stage today.
Connections:
- net 3.3V: no longer U3.27 (SPEED_WAKE)
- new net PWM: U3.27 (SPEED_WAKE)
Changed lines of the file:
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@@
-	)
-	(junction
-		(at 81.28 43.18)
-		(diameter 0)
-		(color 0 0 0 0)
 	)
 	(junction
@@
 	(wire
 		(pts
-			(xy 81.28 43.18) (xy 81.28 48.26)
-		)
-		(stroke
-			(width 0)
-			(type default)
-		)
-	)
-	(wire
-		(pts
 			(xy 181.61 74.93) (xy 185.42 74.93)
 		)
@@
 		(pts
 			(xy 236.22 102.87) (xy 238.76 102.87)
+		)
+		(stroke
+			(width 0)
+			(type default)
+		)
+	)
+	(wire
+		(pts
+			(xy 80.01 48.26) (xy 81.28 48.26)
 		)
 		(stroke
@@
 		(effects
 			(font
+				(size 1.27 1.27)
+			)
+			(justify right)
+		)
+	)
+	(hierarchical_label "PWM"
+		(shape input)
+		(at 80.01 48.26 180)
+		(effects
+			(font

Commit message: I added a green LED.
Parts:
- renumbered C21 to C, C6 to C, C14 to C, C8 to C, C2 to C, C4 to C, C1 to C, C11 to C, C19 to C, C20 to C, Q7 to Q, R9 to R, R6 to R, R3 to R, U3 to U
Connections:
- net SCL renamed I2C_SCL
- net SDA renamed I2C_SDA

Commit message: I added in addressable LEDs, the accelerometers, and some inputs from a receiver just in case.
Parts:
- renumbered C to C12, C to C13, C to C16, C to C17, C to C18, C to C24, C to C25, C to C26, C to C3, C to C5, Q to Q1, R to R16, R to R17, R to R8, U to U5
Changed lines of the file:
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@@
 		(dnp no)
 		(fields_autoplaced yes)
-		(property "Reference" "C"
+		(property "Reference" "C?"
 			(at 57.15 39.3699 0)
 			(effects
@@
 					(unit 1)
 				)
+				(path "/af956454-8f11-4118-89f4-dd7ed925536a/e23ac6b0-b609-49ba-bf9d-eb3b2446a8d3"
+					(reference "C?")
+					(unit 1)
+				)
 			)
 		)
@@
 		(dnp no)
 		(fields_autoplaced yes)
-		(property "Reference" "C"
+		(property "Reference" "C?"
 			(at 45.72 39.3699 0)
 			(effects
@@
 					(unit 1)
 				)
+				(path "/af956454-8f11-4118-89f4-dd7ed925536a/e23ac6b0-b609-49ba-bf9d-eb3b2446a8d3"
+					(reference "C?")
+					(unit 1)
+				)
 			)
 		)
@@
 		(on_board yes)
 		(dnp no)
-		(property "Reference" "Q"
+		(property "Reference" "Q?"
 			(at 160.02 31.7499 90)
 			(effects
@@
 					(unit 1)
 				)
+				(path "/af956454-8f11-4118-89f4-dd7ed925536a/e23ac6b0-b609-49ba-bf9d-eb3b2446a8d3"
+					(reference "Q?")
+					(unit 1)
+				)
 			)
 		)
@@
 		(dnp no)
 		(fields_autoplaced yes)
-		(property "Reference" "C"
+		(property "Reference" "C?"
 			(at 146.05 38.0999 0)
 			(effects
@@
 					(unit 1)
 				)
+				(path "/af956454-8f11-4118-89f4-dd7ed925536a/e23ac6b0-b609-49ba-bf9d-eb3b2446a8d3"
+					(reference "C?")
+					(unit 1)
+				)
 			)
 		)
@@
 		(dnp no)
 		(fields_autoplaced yes)
-		(property "Reference" "C"
+		(property "Reference" "C?"
 			(at 36.83 36.8299 0)
 			(effects
@@
 					(unit 1)
 				)
+				(path "/af956454-8f11-4118-89f4-dd7ed925536a/e23ac6b0-b609-49ba-bf9d-eb3b2446a8d3"
+					(reference "C?")
+					(unit 1)
+				)
 			)
 		)
@@
 		(dnp no)
 		(fields_autoplaced yes)
-		(property "Reference" "C"
+		(property "Reference" "C?"
 			(at 27.94 34.2899 0)
 			(effects
@@
 					(unit 1)
 				)
+				(path "/af956454-8f11-4118-89f4-dd7ed925536a/e23ac6b0-b609-49ba-bf9d-eb3b2446a8d3"
+					(reference "C?")
+					(unit 1)
+				)
 			)
 		)
@@
 		(dnp no)
 		(fields_autoplaced yes)
-		(property "Reference" "C"
+		(property "Reference" "C?"
 			(at 143.51 27.9399 0)
 			(effects
@@
 					(unit 1)
 				)
+				(path "/af956454-8f11-4118-89f4-dd7ed925536a/e23ac6b0-b609-49ba-bf9d-eb3b2446a8d3"
+					(reference "C?")
+					(unit 1)
+				)
 			)
 		)
@@
 		(dnp no)
 		(fields_autoplaced yes)
-		(property "Reference" "C"
+		(property "Reference" "C?"
 			(at 17.78 31.7499 0)
 			(effects
@@
 					(unit 1)
 				)
+				(path "/af956454-8f11-4118-89f4-dd7ed925536a/e23ac6b0-b609-49ba-bf9d-eb3b2446a8d3"
+					(reference "C?")
+					(unit 1)
+				)
 			)
 		)
@@
 		(dnp no)
 		(fields_autoplaced yes)
-		(property "Reference" "C"
+		(property "Reference" "C?"
 			(at 71.12 44.4499 0)
 			(effects
@@
 					(unit 1)
 				)
+				(path "/af956454-8f11-4118-89f4-dd7ed925536a/e23ac6b0-b609-49ba-bf9d-eb3b2446a8d3"
+					(reference "C?")
+					(unit 1)
+				)
 			)
 		)
@@
 		(on_board yes)
 		(dnp no)
-		(property "Reference" "R"
+		(property "Reference" "R?"
 			(at 72.39 86.106 90)
 			(effects
@@
 					(unit 1)
 				)
+				(path "/af956454-8f11-4118-89f4-dd7ed925536a/e23ac6b0-b609-49ba-bf9d-eb3b2446a8d3"
+					(reference "R?")
+					(unit 1)
+				)
 			)
 		)
@@
 		(on_board yes)
 		(dnp no)
-		(property "Reference" "R"
+		(property "Reference" "R?"
 			(at 143.764 170.18 90)
 			(effects
@@
 					(unit 1)
 				)
+				(path "/af956454-8f11-4118-89f4-dd7ed925536a/e23ac6b0-b609-49ba-bf9d-eb3b2446a8d3"
+					(reference "R?")
+					(unit 1)
+				)
 			)
 		)
@@
 		(dnp no)
 		(fields_autoplaced yes)
-		(property "Reference" "C"
+		(property "Reference" "C?"
 			(at 149.86 78.7399 0)
 			(effects
@@
 					(unit 1)
 				)
+				(path "/af956454-8f11-4118-89f4-dd7ed925536a/e23ac6b0-b609-49ba-bf9d-eb3b2446a8d3"
+					(reference "C?")
+					(unit 1)
+				)
 			)
 		)
@@
 		(dnp no)
 		(fields_autoplaced yes)
-		(property "Reference" "C"
+		(property "Reference" "C?"
 			(at 148.59 120.6499 0)
 			(effects
@@
 					(unit 1)
 				)
+				(path "/af956454-8f11-4118-89f4-dd7ed925536a/e23ac6b0-b609-49ba-bf9d-eb3b2446a8d3"
+					(reference "C?")
+					(unit 1)
+				)
 			)
 		)
@@
 		(dnp no)
 		(fields_autoplaced yes)
-		(property "Reference" "R"
+		(property "Reference" "R?"
 			(at 72.39 69.85 90)
 			(effects
@@
 					(unit 1)
 				)
+				(path "/af956454-8f11-4118-89f4-dd7ed925536a/e23ac6b0-b609-49ba-bf9d-eb3b2446a8d3"
+					(reference "R?")
+					(unit 1)
+				)
 			)
 		)
@@
 		(dnp no)
 		(fields_autoplaced yes)
-		(property "Reference" "U"
+		(property "Reference" "U?"
 			(at 109.22 20.32 0)
 			(effects
@@
 					(unit 1)
 				)
+				(path "/af956454-8f11-4118-89f4-dd7ed925536a/e23ac6b0-b609-49ba-bf9d-eb3b2446a8d3"
+					(reference "U?")
+					(unit 1)
+				)

Commit message: I added in the XT30 Connectors for the batteries
Parts:
- renumbered C5 to C11, C12 to C14, C13 to C19, C16 to C20, C17 to C21, C18 to C27, C24 to C28, C25 to C29, C26 to C30, C3 to C8, Q1 to Q7, R17 to R18, R8 to R6, R16 to R9, U5 to U3
Changed lines of the file:
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@@
 		(dnp no)
 		(fields_autoplaced yes)
-		(property "Reference" "C?"
+		(property "Reference" "C20"
 			(at 57.15 39.3699 0)
 			(effects
@@
 				)
 				(path "/af956454-8f11-4118-89f4-dd7ed925536a/e23ac6b0-b609-49ba-bf9d-eb3b2446a8d3"
-					(reference "C?")
+					(reference "C20")
 					(unit 1)
 				)
@@
 		(dnp no)
 		(fields_autoplaced yes)
-		(property "Reference" "C?"
+		(property "Reference" "C19"
 			(at 45.72 39.3699 0)
 			(effects
@@
 				)
 				(path "/af956454-8f11-4118-89f4-dd7ed925536a/e23ac6b0-b609-49ba-bf9d-eb3b2446a8d3"
-					(reference "C?")
+					(reference "C19")
 					(unit 1)
 				)
@@
 		(on_board yes)
 		(dnp no)
-		(property "Reference" "Q?"
+		(property "Reference" "Q7"
 			(at 160.02 31.7499 90)
 			(effects
@@
 				)
 				(path "/af956454-8f11-4118-89f4-dd7ed925536a/e23ac6b0-b609-49ba-bf9d-eb3b2446a8d3"
-					(reference "Q?")
+					(reference "Q7")
 					(unit 1)
 				)
@@
 		(dnp no)
 		(fields_autoplaced yes)
-		(property "Reference" "C?"
+		(property "Reference" "C28"
 			(at 146.05 38.0999 0)
 			(effects
@@
 				)
 				(path "/af956454-8f11-4118-89f4-dd7ed925536a/e23ac6b0-b609-49ba-bf9d-eb3b2446a8d3"
-					(reference "C?")
+					(reference "C28")
 					(unit 1)
 				)
@@
 		(dnp no)
 		(fields_autoplaced yes)
-		(property "Reference" "C?"
+		(property "Reference" "C14"
 			(at 36.83 36.8299 0)
 			(effects
@@
 				)
 				(path "/af956454-8f11-4118-89f4-dd7ed925536a/e23ac6b0-b609-49ba-bf9d-eb3b2446a8d3"
-					(reference "C?")
+					(reference "C14")
 					(unit 1)
 				)
@@
 		(dnp no)
 		(fields_autoplaced yes)
-		(property "Reference" "C?"
+		(property "Reference" "C11"
 			(at 27.94 34.2899 0)
 			(effects
@@
 				)
 				(path "/af956454-8f11-4118-89f4-dd7ed925536a/e23ac6b0-b609-49ba-bf9d-eb3b2446a8d3"
-					(reference "C?")
+					(reference "C11")
 					(unit 1)
 				)
@@
 		(dnp no)
 		(fields_autoplaced yes)
-		(property "Reference" "C?"
+		(property "Reference" "C27"
 			(at 143.51 27.9399 0)
 			(effects
@@
 				)
 				(path "/af956454-8f11-4118-89f4-dd7ed925536a/e23ac6b0-b609-49ba-bf9d-eb3b2446a8d3"
-					(reference "C?")
+					(reference "C27")
 					(unit 1)
 				)
@@
 		(dnp no)
 		(fields_autoplaced yes)
-		(property "Reference" "C?"
+		(property "Reference" "C8"
 			(at 17.78 31.7499 0)
 			(effects
@@
 				)
 				(path "/af956454-8f11-4118-89f4-dd7ed925536a/e23ac6b0-b609-49ba-bf9d-eb3b2446a8d3"
-					(reference "C?")
+					(reference "C8")
 					(unit 1)
 				)
@@
 		(dnp no)
 		(fields_autoplaced yes)
-		(property "Reference" "C?"
+		(property "Reference" "C21"
 			(at 71.12 44.4499 0)
 			(effects
@@
 				)
 				(path "/af956454-8f11-4118-89f4-dd7ed925536a/e23ac6b0-b609-49ba-bf9d-eb3b2446a8d3"
-					(reference "C?")
+					(reference "C21")
 					(unit 1)
 				)
@@
 		(on_board yes)
 		(dnp no)
-		(property "Reference" "R?"
+		(property "Reference" "R9"
 			(at 72.39 86.106 90)
 			(effects
@@
 				)
 				(path "/af956454-8f11-4118-89f4-dd7ed925536a/e23ac6b0-b609-49ba-bf9d-eb3b2446a8d3"
-					(reference "R?")
+					(reference "R9")
 					(unit 1)
 				)
@@
 		(on_board yes)
 		(dnp no)
-		(property "Reference" "R?"
+		(property "Reference" "R18"
 			(at 143.764 170.18 90)
 			(effects
@@
 				)
 				(path "/af956454-8f11-4118-89f4-dd7ed925536a/e23ac6b0-b609-49ba-bf9d-eb3b2446a8d3"
-					(reference "R?")
+					(reference "R18")
 					(unit 1)
 				)
@@
 		(dnp no)
 		(fields_autoplaced yes)
-		(property "Reference" "C?"
+		(property "Reference" "C30"
 			(at 149.86 78.7399 0)
 			(effects
@@
 				)
 				(path "/af956454-8f11-4118-89f4-dd7ed925536a/e23ac6b0-b609-49ba-bf9d-eb3b2446a8d3"
-					(reference "C?")
+					(reference "C30")
 					(unit 1)
 				)
@@
 		(dnp no)
 		(fields_autoplaced yes)
-		(property "Reference" "C?"
+		(property "Reference" "C29"
 			(at 148.59 120.6499 0)
 			(effects
@@
 				)
 				(path "/af956454-8f11-4118-89f4-dd7ed925536a/e23ac6b0-b609-49ba-bf9d-eb3b2446a8d3"
-					(reference "C?")
+					(reference "C29")
 					(unit 1)
 				)
@@
 		(dnp no)
 		(fields_autoplaced yes)
-		(property "Reference" "R?"
+		(property "Reference" "R6"
 			(at 72.39 69.85 90)
 			(effects
@@
 				)
 				(path "/af956454-8f11-4118-89f4-dd7ed925536a/e23ac6b0-b609-49ba-bf9d-eb3b2446a8d3"
-					(reference "R?")
+					(reference "R6")
 					(unit 1)
 				)
@@
 		(dnp no)
 		(fields_autoplaced yes)
-		(property "Reference" "U?"
+		(property "Reference" "U3"
 			(at 109.22 20.32 0)
 			(effects
@@
 				)
 				(path "/af956454-8f11-4118-89f4-dd7ed925536a/e23ac6b0-b609-49ba-bf9d-eb3b2446a8d3"
-					(reference "U?")
+					(reference "U3")
 					(unit 1)
 				)

Commit message: fixed all the schematic errors.
Parts:
- added J8: MR30PW-FB, Footprints:MR30PWFB, symbol MR30PW-FB:MR30PW-FB
- C10: renamed from C19; Stock 1647341 -> 1551376
- C11: renamed from C20; Stock 64667839 -> 58347526
- C12: renamed from C21; Stock 17190513 -> 16297537
- C13: renamed from C27; Stock 676425 -> 611581
- C14: renamed from C28; Stock 17190513 -> 16297537
- C15: renamed from C29; Stock 17190513 -> 16297537
- C16: renamed from C30; Stock 17190513 -> 16297537
- C7: renamed from C8; Stock 17190513 -> 16297537
- C8: renamed from C11; Stock 17190513 -> 16297537
- C9: renamed from C14; Stock 1647341 -> 1551376
- Q2: renamed from Q8; footprint NVMFS5C442NLWFAFT1G -> Footprints:NVMFS5C442NLWFAFT1G
- Q3: renamed from Q9; footprint NVMFS5C442NLWFAFT1G -> Footprints:NVMFS5C442NLWFAFT1G
- Q4: renamed from Q10; footprint NVMFS5C442NLWFAFT1G -> Footprints:NVMFS5C442NLWFAFT1G
- Q5: renamed from Q11; footprint NVMFS5C442NLWFAFT1G -> Footprints:NVMFS5C442NLWFAFT1G
- Q6: renamed from Q12; footprint NVMFS5C442NLWFAFT1G -> Footprints:NVMFS5C442NLWFAFT1G
- R10: renamed from R6; Stock 17848646 -> 16030120
- R11: renamed from R10; Stock 4532170 -> 4254023
- R12: renamed from R9; Stock 4532170 -> 4254023
- R9: renamed from R4; Stock 17848646 -> 16030120
- renumbered Q7 to Q1, R18 to R13, U3 to U4
Connections:
- net 3.3V is gone; now on net +3.3V: C12.1, U4.2 (VREG)
- net PhaseB: now reaches Q3.1 (S_1), Q3.2 (S_2), Q3.3 (S_3), Q4.5 (D_1), Q4.6 (D_2), Q4.7 (D_3), Q4.8 (D_4), Q4.9 (D_5)
- net PhaseB: now also J8.2
- net PhaseC: now reaches Q5.1 (S_1), Q5.2 (S_2), Q5.3 (S_3), Q6.5 (D_1), Q6.6 (D_2), Q6.7 (D_3), Q6.8 (D_4), Q6.9 (D_5)
- net PhaseC: now also J8.3
- net PhaseA: now reaches C14.2, Q1.1 (S_1), Q1.2 (S_2), Q1.3 (S_3), Q2.5 (D_1), Q2.6 (D_2), Q2.7 (D_3), Q2.8 (D_4), Q2.9 (D_5), U4.10 (SHA)
- net PhaseA: now also J8.1
- no-connect marks 3 -> 5
