File: OmniAnt/H3LIS331DL.kicad_sch (KiCad schematic)
At the start: 3 parts

Commit message: I added in the XT30 Connectors for the batteries
Parts:
- renumbered AC to AC1
Changed lines of the file:
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@@
 		(on_board yes)
 		(dnp no)
-		(property "Reference" "AC"
+		(property "Reference" "AC1"
 			(at 119.38 106.934 0)
 			(effects
@@
 					(unit 1)
 				)
+				(path "/af956454-8f11-4118-89f4-dd7ed925536a/715d742c-13c6-4f25-8121-09fc2df5f196"
+					(reference "AC1")
+					(unit 1)
+				)

Commit message: fixed all the schematic errors.
Parts:
- C27: renamed from C2; Stock 64667839 -> 58347526
- C28: renamed from C1; Stock 1647341 -> 1551376
Connections:
- net GND: now also AC1.10 (RESERVED_1), AC1.12 (GND_2), AC1.13 (GND_3), C27.2, C28.2
Changed lines of the file:
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@@
 	(paper "A4")
+	(junction
+		(at 128.27 82.55)
+		(diameter 0)
+		(color 0 0 0 0)
+	)
+	(junction
+		(at 82.55 85.09)
+		(diameter 0)
+		(color 0 0 0 0)
+	)
+	(junction
+		(at 82.55 74.93)
+		(diameter 0)
+		(color 0 0 0 0)
+	)
 	(junction
 		(at 128.27 74.93)
@@
 	(wire
 		(pts
+			(xy 74.93 85.09) (xy 82.55 85.09)
+		)
+		(stroke
+			(width 0)
+			(type default)
+		)
+	)
+	(wire
+		(pts
 			(xy 128.27 77.47) (xy 123.19 77.47)
 		)
@@
 	(wire
 		(pts
+			(xy 74.93 74.93) (xy 82.55 74.93)
+		)
+		(stroke
+			(width 0)
+			(type default)
+		)
+	)
+	(wire
+		(pts
 			(xy 123.19 82.55) (xy 128.27 82.55)
 		)
@@
 			(width 0)
 			(type default)
+		)
+	)
+	(hierarchical_label "+3.3V"
+		(shape input)
+		(at 74.93 74.93 180)
+		(effects
+			(font
+				(size 1.27 1.27)
+			)
+			(justify right)
 		)
 	)
@@
 		)
 	)
+	(hierarchical_label "GND"
+		(shape input)
+		(at 74.93 85.09 180)
+		(effects
+			(font
+				(size 1.27 1.27)
+			)
+			(justify right)
+		)
+	)
 	(hierarchical_label "SPI_MOSI"
 		(shape input)
@@
 			)
 			(justify left)
+		)
+	)
+	(symbol
+		(lib_id "power:GND")
+		(at 128.27 82.55 0)
+		(unit 1)
+		(exclude_from_sim no)
+		(in_bom yes)
+		(on_board yes)
+		(dnp no)
+		(fields_autoplaced yes)
+		(property "Reference" "#PWR034"
+			(at 128.27 88.9 0)
+			(effects
+				(font
+					(size 1.27 1.27)
+				)
+				(hide yes)
+			)
+		)
+		(property "Value" "GND"
+			(at 128.27 87.63 0)
+			(effects
+				(font
+					(size 1.27 1.27)
+				)
+			)
+		)
+		(property "Footprint" ""
+			(at 128.27 82.55 0)
+			(effects
+				(font
+					(size 1.27 1.27)
+				)
+				(hide yes)
+			)
+		)
+		(property "Datasheet" ""
+			(at 128.27 82.55 0)
+			(effects
+				(font
+					(size 1.27 1.27)
+				)
+				(hide yes)
+			)
+		)
+		(property "Description" "Power symbol creates a global label with name \"GND\" , ground"
+			(at 128.27 82.55 0)
+			(effects
+				(font
+					(size 1.27 1.27)
+				)
+				(hide yes)
+			)
+		)
+		(pin "1"
+		)
+		(instances
+			(project "OmniAnt"
+				(path "/af956454-8f11-4118-89f4-dd7ed925536a/26834c6c-f4a8-48a9-9b9e-c769f479a855"
+					(reference "#PWR039")
+					(unit 1)
+				)
+				(path "/af956454-8f11-4118-89f4-dd7ed925536a/715d742c-13c6-4f25-8121-09fc2df5f196"
+					(reference "#PWR034")
+					(unit 1)
+				)
+			)
 		)
 	)
@@
 		(dnp no)
 		(fields_autoplaced yes)
-		(property "Reference" "#PWR020"
+		(property "Reference" "#PWR031"
 			(at 82.55 95.25 0)
 			(effects
@@
 		(instances
 			(project "OmniAnt"
-				(path "/af956454-8f11-4118-89f4-dd7ed925536a/495e6d06-414b-4f15-a3c9-6bced6a7e482"
-					(reference "#PWR025")
+				(path "/af956454-8f11-4118-89f4-dd7ed925536a/26834c6c-f4a8-48a9-9b9e-c769f479a855"
+					(reference "#PWR036")
 					(unit 1)
 				)
 				(path "/af956454-8f11-4118-89f4-dd7ed925536a/715d742c-13c6-4f25-8121-09fc2df5f196"
-					(reference "#PWR020")
+					(reference "#PWR031")
 					(unit 1)
 				)
@@
 		(instances
 			(project "OmniAnt"
-				(path "/af956454-8f11-4118-89f4-dd7ed925536a/495e6d06-414b-4f15-a3c9-6bced6a7e482"
+				(path "/af956454-8f11-4118-89f4-dd7ed925536a/26834c6c-f4a8-48a9-9b9e-c769f479a855"
 					(reference "AC2")
 					(unit 1)
@@
 		(on_board yes)
 		(dnp no)
-		(property "Reference" "#PWR022"
+		(property "Reference" "#PWR030"
 			(at 82.55 78.74 0)
 			(effects
@@
 		(instances
 			(project "OmniAnt"
-				(path "/af956454-8f11-4118-89f4-dd7ed925536a/495e6d06-414b-4f15-a3c9-6bced6a7e482"
-					(reference "#PWR024")
+				(path "/af956454-8f11-4118-89f4-dd7ed925536a/26834c6c-f4a8-48a9-9b9e-c769f479a855"
+					(reference "#PWR035")
 					(unit 1)
 				)
 				(path "/af956454-8f11-4118-89f4-dd7ed925536a/715d742c-13c6-4f25-8121-09fc2df5f196"
-					(reference "#PWR022")
+					(reference "#PWR030")
 					(unit 1)
 				)
@@
 		(dnp no)
 		(fields_autoplaced yes)
-		(property "Reference" "C1"
+		(property "Reference" "C28"
 			(at 134.62 53.3399 0)
 			(effects
@@
 			)
 		)
-		(property "Stock" "1647341"
+		(property "Stock" "1551376"
 			(at 132.08 55.88 0)
 			(effects
@@
 		(instances
 			(project "OmniAnt"
-				(path "/af956454-8f11-4118-89f4-dd7ed925536a/495e6d06-414b-4f15-a3c9-6bced6a7e482"
-					(reference "C6")
+				(path "/af956454-8f11-4118-89f4-dd7ed925536a/26834c6c-f4a8-48a9-9b9e-c769f479a855"
+					(reference "C30")
 					(unit 1)
 				)
 				(path "/af956454-8f11-4118-89f4-dd7ed925536a/715d742c-13c6-4f25-8121-09fc2df5f196"
-					(reference "C1")
+					(reference "C28")
 					(unit 1)
 				)
@@
 		(dnp no)
 		(fields_autoplaced yes)
-		(property "Reference" "C2"
+		(property "Reference" "C27"
 			(at 125.73 53.3399 0)
 			(effects
@@
 			)
 		)
-		(property "Stock" "64667839"
+		(property "Stock" "58347526"
 			(at 123.19 55.88 0)
 			(effects
@@
 		(instances
 			(project "OmniAnt"
-				(path "/af956454-8f11-4118-89f4-dd7ed925536a/495e6d06-414b-4f15-a3c9-6bced6a7e482"
-					(reference "C4")
+				(path "/af956454-8f11-4118-89f4-dd7ed925536a/26834c6c-f4a8-48a9-9b9e-c769f479a855"
+					(reference "C29")
 					(unit 1)
 				)
 				(path "/af956454-8f11-4118-89f4-dd7ed925536a/715d742c-13c6-4f25-8121-09fc2df5f196"
-					(reference "C2")
+					(reference "C27")
 					(unit 1)
 				)
@@
 		(dnp no)
 		(fields_autoplaced yes)
-		(property "Reference" "#PWR023"
+		(property "Reference" "#PWR032"
 			(at 83.82 64.77 0)
 			(effects
@@
 		(instances
 			(project "OmniAnt"
-				(path "/af956454-8f11-4118-89f4-dd7ed925536a/495e6d06-414b-4f15-a3c9-6bced6a7e482"
-					(reference "#PWR026")
+				(path "/af956454-8f11-4118-89f4-dd7ed925536a/26834c6c-f4a8-48a9-9b9e-c769f479a855"
+					(reference "#PWR037")
 					(unit 1)
 				)
 				(path "/af956454-8f11-4118-89f4-dd7ed925536a/715d742c-13c6-4f25-8121-09fc2df5f196"
-					(reference "#PWR023")
+					(reference "#PWR032")
 					(unit 1)
 				)
@@
 		(on_board yes)
 		(dnp no)
-		(property "Reference" "#PWR021"
+		(property "Reference" "#PWR033"
 			(at 105.41 53.34 0)
 			(effects
@@
 		(instances
 			(project "OmniAnt"
-				(path "/af956454-8f11-4118-89f4-dd7ed925536a/495e6d06-414b-4f15-a3c9-6bced6a7e482"
-					(reference "#PWR027")
+				(path "/af956454-8f11-4118-89f4-dd7ed925536a/26834c6c-f4a8-48a9-9b9e-c769f479a855"
+					(reference "#PWR038")
 					(unit 1)
 				)
 				(path "/af956454-8f11-4118-89f4-dd7ed925536a/715d742c-13c6-4f25-8121-09fc2df5f196"
-					(reference "#PWR021")
-					(unit 1)
-				)
+					(reference "#PWR033")
+					(unit 1)
+				)

Commit message: Well shit making the FETs into libraries totally screwed up the annotation :( I decided to just redo the layout for the FETs anyhow.
Parts:
- C401: renamed from C27; Stock 58347526 -> 64667839
- C402: renamed from C28; Stock 1551376 -> 1647341
- renumbered AC1 to AC401
Changed lines of the file:
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@@
 		(dnp no)
 		(fields_autoplaced yes)
-		(property "Reference" "#PWR034"
+		(property "Reference" "#PWR0405"
 			(at 128.27 88.9 0)
 			(effects
@@
 			(project "OmniAnt"
 				(path "/af956454-8f11-4118-89f4-dd7ed925536a/26834c6c-f4a8-48a9-9b9e-c769f479a855"
-					(reference "#PWR039")
+					(reference "#PWR0505")
 					(unit 1)
 				)
 				(path "/af956454-8f11-4118-89f4-dd7ed925536a/715d742c-13c6-4f25-8121-09fc2df5f196"
-					(reference "#PWR034")
+					(reference "#PWR0405")
 					(unit 1)
 				)
@@
 		(dnp no)
 		(fields_autoplaced yes)
-		(property "Reference" "#PWR031"
+		(property "Reference" "#PWR0402"
 			(at 82.55 95.25 0)
 			(effects
@@
 			(project "OmniAnt"
 				(path "/af956454-8f11-4118-89f4-dd7ed925536a/26834c6c-f4a8-48a9-9b9e-c769f479a855"
-					(reference "#PWR036")
+					(reference "#PWR0502")
 					(unit 1)
 				)
 				(path "/af956454-8f11-4118-89f4-dd7ed925536a/715d742c-13c6-4f25-8121-09fc2df5f196"
-					(reference "#PWR031")
+					(reference "#PWR0402")
 					(unit 1)
 				)
@@
 		(on_board yes)
 		(dnp no)
-		(property "Reference" "AC1"
+		(property "Reference" "AC401"
 			(at 119.38 106.934 0)
 			(effects
@@
 			(project "OmniAnt"
 				(path "/af956454-8f11-4118-89f4-dd7ed925536a/26834c6c-f4a8-48a9-9b9e-c769f479a855"
-					(reference "AC2")
+					(reference "AC501")
 					(unit 1)
 				)
 				(path "/af956454-8f11-4118-89f4-dd7ed925536a/715d742c-13c6-4f25-8121-09fc2df5f196"
-					(reference "AC1")
+					(reference "AC401")
 					(unit 1)
 				)
@@
 		(on_board yes)
 		(dnp no)
-		(property "Reference" "#PWR030"
+		(property "Reference" "#PWR0401"
 			(at 82.55 78.74 0)
 			(effects
@@
 			(project "OmniAnt"
 				(path "/af956454-8f11-4118-89f4-dd7ed925536a/26834c6c-f4a8-48a9-9b9e-c769f479a855"
-					(reference "#PWR035")
+					(reference "#PWR0501")
 					(unit 1)
 				)
 				(path "/af956454-8f11-4118-89f4-dd7ed925536a/715d742c-13c6-4f25-8121-09fc2df5f196"
-					(reference "#PWR030")
+					(reference "#PWR0401")
 					(unit 1)
 				)
@@
 		(dnp no)
 		(fields_autoplaced yes)
-		(property "Reference" "C28"
+		(property "Reference" "C402"
 			(at 134.62 53.3399 0)
 			(effects
@@
 			)
 		)
-		(property "Stock" "1551376"
+		(property "Stock" "1647341"
 			(at 132.08 55.88 0)
 			(effects
@@
 			(project "OmniAnt"
 				(path "/af956454-8f11-4118-89f4-dd7ed925536a/26834c6c-f4a8-48a9-9b9e-c769f479a855"
-					(reference "C30")
+					(reference "C502")
 					(unit 1)
 				)
 				(path "/af956454-8f11-4118-89f4-dd7ed925536a/715d742c-13c6-4f25-8121-09fc2df5f196"
-					(reference "C28")
+					(reference "C402")
 					(unit 1)
 				)
@@
 		(dnp no)
 		(fields_autoplaced yes)
-		(property "Reference" "C27"
+		(property "Reference" "C401"
 			(at 125.73 53.3399 0)
 			(effects
@@
 			)
 		)
-		(property "Stock" "58347526"
+		(property "Stock" "64667839"
 			(at 123.19 55.88 0)
 			(effects
@@
 			(project "OmniAnt"
 				(path "/af956454-8f11-4118-89f4-dd7ed925536a/26834c6c-f4a8-48a9-9b9e-c769f479a855"
-					(reference "C29")
+					(reference "C501")
 					(unit 1)
 				)
 				(path "/af956454-8f11-4118-89f4-dd7ed925536a/715d742c-13c6-4f25-8121-09fc2df5f196"
-					(reference "C27")
+					(reference "C401")
 					(unit 1)
 				)
@@
 		(dnp no)
 		(fields_autoplaced yes)
-		(property "Reference" "#PWR032"
+		(property "Reference" "#PWR0403"
 			(at 83.82 64.77 0)
 			(effects
@@
 			(project "OmniAnt"
 				(path "/af956454-8f11-4118-89f4-dd7ed925536a/26834c6c-f4a8-48a9-9b9e-c769f479a855"
-					(reference "#PWR037")
+					(reference "#PWR0503")
 					(unit 1)
 				)
 				(path "/af956454-8f11-4118-89f4-dd7ed925536a/715d742c-13c6-4f25-8121-09fc2df5f196"
-					(reference "#PWR032")
+					(reference "#PWR0403")
 					(unit 1)
 				)
@@
 		(on_board yes)
 		(dnp no)
-		(property "Reference" "#PWR033"
+		(property "Reference" "#PWR0404"
 			(at 105.41 53.34 0)
 			(effects
@@
 			(project "OmniAnt"
 				(path "/af956454-8f11-4118-89f4-dd7ed925536a/26834c6c-f4a8-48a9-9b9e-c769f479a855"
-					(reference "#PWR038")
+					(reference "#PWR0504")
 					(unit 1)
 				)
 				(path "/af956454-8f11-4118-89f4-dd7ed925536a/715d742c-13c6-4f25-8121-09fc2df5f196"
-					(reference "#PWR033")
-					(unit 1)
-				)
+					(reference "#PWR0404")
+					(unit 1)
+				)
