File: OmniAnt/OmniAnt.kicad_pcb (KiCad board)
At the start: 4 copper layers, 228 parts, among them J101 Connector, USB-TYPE-C-16P, J102 Conn_01x02_Pin, J103 Conn_01x04_Pin, J104 Conn_01x02_Pin, J105 Conn_01x02_Pin, J106 XT30PW-M, J107 XT30PW-M, J108 XT30PW-M, J109 XT30PW-M, J110 Conn_01x01, J111 Conn_01x01, J112 Conn_01x01, J113 Conn_01x01, J114 Conn_01x01, J115 Conn_01x01, J116 Conn_01x01, J117 Conn_01x01, J118 Conn_01x01, J119 Conn_01x01, J201 Conn_01x01, J202 Conn_01x01, J203 Conn_01x01, J204 Conn_01x01, J205 Conn_01x01, J206 Conn_01x01, J207 Conn_01x01, J208 Conn_01x01, J209 Conn_01x01, J210 Conn_01x01, J211 Conn_01x01, J301 Conn_01x01, J302 Conn_01x01, J303 Conn_01x01, J304 Conn_01x01, J305 Conn_01x01, J306 Conn_01x01, J307 Conn_01x01, J308 Conn_01x01, J309 Conn_01x01, J310 Conn_01x01, J311 Conn_01x01, Q1101 NTMFS4C324NT1G, Q1201 NTMFS4C324NT1G, Q1501 NTMFS4C324NT1G, Q1601 NTMFS4C324NT1G, Q1701 NTMFS4C324NT1G, Q801 NTMFS4C324NT1G, U101 USBLC6-2P6, U102 TPSM53603RDA, U103 ESP32-S3-WROOM-1, U201 MCF8329A1IREER, U301 MCF8329A1IREER

Commit message: Really good progress. I positioned everything, and ran a bunch of signals.
Parts:
- removed the R101 at (233.2, 32.2)
- removed the R102 at (236.2, 32.2)
- J101: value Connector, USB-TYPE-C-16P -> USB_B_Micro; footprint PCM_JLCPCB:TYPE-C-SMD_HX-TYPE-C-16PIN -> Connector_USB:USB_Micro-B_Molex-105017-0001
- moved Q1301 172.8 mm to (138.3, 43.1), turned to 90 degrees
- moved D1302 171.3 mm to (144.3, 42.3), turned to -90 degrees
- moved R1303 170.9 mm to (146.5, 41.4), turned to -90 degrees
- moved D1301 169.1 mm to (147.7, 39.5), turned to 180 degrees
- moved D1303 168.3 mm to (140.1, 48.6), turned to 180 degrees
- moved Q901 167.8 mm to (138.4, 29.2), turned to 90 degrees
- moved D902 166.8 mm to (144.4, 28.4), turned to -90 degrees
- moved D903 164.4 mm to (140.1, 34.7), turned to 180 degrees
- moved R903 164.1 mm to (146.5, 27.5), turned to -90 degrees
- moved Q701 163.0 mm to (123.0, 14.6), turned to 90 degrees
- moved D901 162.7 mm to (147.7, 25.5), turned to 180 degrees
- moved D702 161.8 mm to (129.0, 13.8), turned to -90 degrees
- moved C1301 161.5 mm to (136.0, 49.4), turned to -90 degrees
- moved R703 159.3 mm to (131.9, 9.09)
- moved C701 159.1 mm to (130.0, 18.7), turned to 90 degrees
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- renumbered QHB1001 to Q1001, QLC1301 to Q1301, QHC1401 to Q1401, QLA601 to Q601, QHA701 to Q701, QLB901 to Q901, R103 to R101, R104 to R102, R105 to R103, R106 to R104, R107 to R105, R108 to R106
Connections:
- U101 pad 1: /D- -> /D+
- U101 pad 3: /D+ -> /D-
- U101 pad 4: Net-(J101-D+-PadA6) -> /USB_D-
- U101 pad 6: Net-(J101-D--PadA7) -> /USB_D+
Routing:
- net /Batt: track 6.85 -> 97.7 mm
- net /D-: track 0.00 -> 77.5 mm
- net /D+: track 0.00 -> 76.9 mm
- net /Motor2_DAC: track 0.00 -> 60.7 mm, vias 0 -> 2
- net /I2C_SCL: track 0.00 -> 59.9 mm, vias 0 -> 1
- net /I2C_SDA: track 0.00 -> 57.9 mm, vias 0 -> 1
- net /Motor2/LSS: track 59.4 -> 4.27 mm
- net /SPI2_CS: track 0.00 -> 50.1 mm, vias 0 -> 2
- net /SPI2_MOSI: track 0.00 -> 34.7 mm, vias 0 -> 2
- net /SPI2_MISO: track 0.00 -> 34.5 mm, vias 0 -> 2
- net /SPI2_SCK: track 0.00 -> 34.5 mm, vias 0 -> 2
- net /Motor1/PhaseA: track 0.00 -> 34.2 mm
- net /Motor2_PWM: track 1.40 -> 35.4 mm, vias 0 -> 1
- net /Accel2_INT: track 0.00 -> 32.4 mm, vias 0 -> 2
- net /Motor1/QHA/G: track 0.00 -> 31.8 mm
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- added copper zone on F.Cu, net +3.3V
- added copper zone on B.Cu, net /Batt_1S
- added copper zone on F.Cu, net /Batt_1S
- added copper zone on In1.Cu, net /Batt_1S
- added copper zone on In2.Cu, net /Batt_1S
- added copper zone on B.Cu, net /Batt_2S
- added copper zone on F.Cu, net /Batt_2S
- added copper zone on In1.Cu, net /Batt_2S
- added copper zone on In2.Cu, net /Batt_2S
- added copper zone on B.Cu, net /Batt_3S
- added copper zone on F.Cu, net /Batt_3S
- added copper zone on In1.Cu, net /Batt_3S
- added copper zone on In2.Cu, net /Batt_3S
- added copper zone on B.Cu, net /Motor1/LSS
- added copper zone on F.Cu, net /Motor1/LSS
- added copper zone on In1.Cu, net /Motor1/LSS
- added copper zone on In2.Cu, net /Motor1/LSS
- added copper zone on B.Cu, net /Motor1/PhaseA
- added copper zone on F.Cu, net /Motor1/PhaseA
- added copper zone on In1.Cu, net /Motor1/PhaseA
- added copper zone on In2.Cu, net /Motor1/PhaseA
- added copper zone on B.Cu, net /Motor1/PhaseB
- added copper zone on F.Cu, net /Motor1/PhaseB
- added copper zone on In1.Cu, net /Motor1/PhaseB
- added copper zone on In2.Cu, net /Motor1/PhaseB
- added copper zone on B.Cu, net /Motor1/PhaseC
- added copper zone on F.Cu, net /Motor1/PhaseC
- added copper zone on In1.Cu, net /Motor1/PhaseC
- added copper zone on In2.Cu, net /Motor1/PhaseC
- added copper zone on F.Cu, net /Motor1/QHA/G
- added copper zone on F.Cu, net /Motor1/QHB/G
- added copper zone on F.Cu, net /Motor1/QHC/G
- added copper zone on F.Cu, net /Motor1/QLA/G
- added copper zone on F.Cu, net /Motor1/QLB/G
- added copper zone on F.Cu, net /Motor1/QLC/G
- added copper zone on B.Cu, net /Motor2/LSS
- added copper zone on F.Cu, net /VUSB
- added copper zone on B.Cu, net GND
- added copper zone on F.Cu, net GND
- added copper zone on In1.Cu, net GND
- added copper zone on In2.Cu, net GND
- added copper zone on B.Cu, net Net-(C1001-Pad1)
- added copper zone on F.Cu, net Net-(C1001-Pad1)
- added copper zone on In1.Cu, net Net-(C1001-Pad1)
- added copper zone on In2.Cu, net Net-(C1001-Pad1)
- added copper zone on B.Cu, net Net-(C1301-Pad1)
- added copper zone on F.Cu, net Net-(C1301-Pad1)
- added copper zone on In1.Cu, net Net-(C1301-Pad1)
- added copper zone on In2.Cu, net Net-(C1301-Pad1)
- added copper zone on B.Cu, net Net-(C601-Pad1)
- added copper zone on F.Cu, net Net-(C601-Pad1)
- added copper zone on In1.Cu, net Net-(C601-Pad1)
- added copper zone on In2.Cu, net Net-(C601-Pad1)
- added copper zone on B.Cu, net Net-(C701-Pad1)
- added copper zone on F.Cu, net Net-(C701-Pad1)
- added copper zone on In1.Cu, net Net-(C701-Pad1)
- added copper zone on In2.Cu, net Net-(C701-Pad1)
- added copper zone on B.Cu, net Net-(C901-Pad1)
- added copper zone on F.Cu, net Net-(C901-Pad1)
- added copper zone on In1.Cu, net Net-(C901-Pad1)
- added copper zone on In2.Cu, net Net-(C901-Pad1)
- added copper zone on B.Cu, net Net-(D1001-Pad1)
- added copper zone on F.Cu, net Net-(D1001-Pad1)
- added copper zone on In1.Cu, net Net-(D1001-Pad1)
- added copper zone on In2.Cu, net Net-(D1001-Pad1)
- added copper zone on B.Cu, net Net-(D1301-Pad1)
- added copper zone on F.Cu, net Net-(D1301-Pad1)
- added copper zone on In1.Cu, net Net-(D1301-Pad1)
- added copper zone on In2.Cu, net Net-(D1301-Pad1)
- added copper zone on B.Cu, net Net-(D1401-Pad1)
- added copper zone on F.Cu, net Net-(D1401-Pad1)
- added copper zone on In1.Cu, net Net-(D1401-Pad1)
- added copper zone on In2.Cu, net Net-(D1401-Pad1)
- added copper zone on B.Cu, net Net-(D601-Pad1)
- added copper zone on F.Cu, net Net-(D601-Pad1)
- added copper zone on In1.Cu, net Net-(D601-Pad1)
- added copper zone on In2.Cu, net Net-(D601-Pad1)
- added copper zone on B.Cu, net Net-(D701-Pad1)
- added copper zone on F.Cu, net Net-(D701-Pad1)
- added copper zone on In1.Cu, net Net-(D701-Pad1)
- added copper zone on In2.Cu, net Net-(D701-Pad1)
- added copper zone on B.Cu, net Net-(D901-Pad1)
- added copper zone on F.Cu, net Net-(D901-Pad1)
- added copper zone on In1.Cu, net Net-(D901-Pad1)
- added copper zone on In2.Cu, net Net-(D901-Pad1)
- added copper zone on F.Cu, net Net-(Q1001-G)
- added copper zone on F.Cu, net Net-(Q1301-G)
- added copper zone on F.Cu, net Net-(Q601-G)
- added copper zone on F.Cu, net Net-(Q701-G)
- added copper zone on F.Cu, net Net-(Q901-G)
- added copper zone on F.Cu, net Net-(U102-FB)
- added copper zone on F.Cu, net Net-(U201-BSTB)
- added copper zone on F.Cu, net Net-(U201-BSTC)
- removed copper zone on B.Cu, net Net-(Q1401-G)
- removed copper zone on In1.Cu, net Net-(Q1401-G)
- removed copper zone on In2.Cu, net Net-(Q1401-G)
Other:
- board outline added: 306.9 x 44.7 mm

Commit message: Everything looks good to me. I'm going to run design checks now. I'm sure it is going to be bad.
Parts:
- added H106: MountingHole, MountingHole:MountingHole_3mm, F.Cu at (46.6, 66.6)
- added H107: MountingHole, MountingHole:MountingHole_3mm, F.Cu at (240.1, 66.6)
- moved U101 105.7 mm to (130.8, 69.9), turned to 90 degrees
- moved J101 104.8 mm to (130.5, 65.9), turned to 180 degrees
- moved D101 102.1 mm to (133.3, 72.4), turned to 90 degrees
- moved C102 102.1 mm to (144.9, 88.7), turned to 0 degrees
- moved C105 101.3 mm to (148.9, 88.8), turned to 180 degrees
- moved J119 101.1 mm to (137.0, 80.3), turned to -90 degrees
- moved C101 100.4 mm to (133.3, 69.0), turned to 0 degrees
- moved AC501 98.1 mm to (153.4, 102.4)
- moved C501 98.1 mm to (154.4, 100.0)
- moved C502 98.1 mm to (154.7, 98.4)
- moved AC401 98.1 mm to (143.4, 92.4)
- moved C401 98.1 mm to (145.8, 93.4)
- moved C402 98.1 mm to (147.4, 93.7)
- moved H103 98.1 mm to (143.4, 102.4)
- moved U102 96.0 mm to (147.0, 84.7), turned to 90 degrees
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Connections:
- R105 pad 1: /I2C_SDA -> /I2C_SCL
- R106 pad 1: /I2C_SCL -> /I2C_SDA
- U103 pad 24: /I2C_SDA -> /I2C_SCL
- U103 pad 25: /I2C_SCL -> /I2C_SDA
- U201 pad 38: (no net) -> GND
- U201 pad 39: (no net) -> GND
- U201 pad 40: (no net) -> GND
- U201 pad 41: (no net) -> GND
- U201 pad 42: (no net) -> GND
- U201 pad 43: (no net) -> GND
- U201 pad 44: (no net) -> GND
- U201 pad 45: (no net) -> GND
- U301 pad 38: (no net) -> GND
- U301 pad 39: (no net) -> GND
- U301 pad 40: (no net) -> GND
- U301 pad 41: (no net) -> GND
- U301 pad 42: (no net) -> GND
- U301 pad 43: (no net) -> GND
- U301 pad 44: (no net) -> GND
- U301 pad 45: (no net) -> GND
Routing:
- net Net-(D102-DIN): track 0.00 -> 182.6 mm
- net /Motor2_PWM: track 35.4 -> 99.5 mm, vias 1 -> 2
- net Net-(D103-DIN): track 0.00 -> 51.4 mm, vias 0 -> 1
- net Net-(U103-IO16): track 0.00 -> 49.6 mm
- net /D+: track 76.9 -> 33.3 mm, vias 0 -> 2
- net /D-: track 77.5 -> 34.3 mm, vias 0 -> 2
- net /Motor1_DAC: track 0.00 -> 38.2 mm, vias 0 -> 2
- net /I2C_SDA: track 57.9 -> 91.9 mm, vias 1 -> 2
- net /I2C_SCL: track 59.9 -> 89.3 mm
- net /Accel1_INT: track 10.6 -> 36.5 mm
- net /SPI1_CS: track 8.13 -> 30.5 mm
- net /SPI2_CS: track 50.1 -> 72.1 mm
- net /Accel2_INT: track 32.4 -> 52.1 mm
- net /SPI1_MISO: track 9.70 -> 29.1 mm
- net /Motor2_DAC: track 60.7 -> 79.0 mm
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- added copper zone on In2.Cu, net +3.3V
- added copper zone on F.Cu, net Net-(U103-EN)
- removed copper zone on B.Cu, net Net-(D1001-Pad1)
- removed copper zone on In1.Cu, net Net-(D1001-Pad1)
- removed copper zone on In2.Cu, net Net-(D1001-Pad1)
- removed copper zone on B.Cu, net Net-(D1101-Pad1)
- removed copper zone on In1.Cu, net Net-(D1101-Pad1)
- removed copper zone on In2.Cu, net Net-(D1101-Pad1)
- removed copper zone on B.Cu, net Net-(D1201-Pad1)
- removed copper zone on In1.Cu, net Net-(D1201-Pad1)
- removed copper zone on In2.Cu, net Net-(D1201-Pad1)
- removed copper zone on B.Cu, net Net-(D1301-Pad1)
- removed copper zone on In1.Cu, net Net-(D1301-Pad1)
- removed copper zone on In2.Cu, net Net-(D1301-Pad1)
- removed copper zone on B.Cu, net Net-(D1401-Pad1)
- removed copper zone on In1.Cu, net Net-(D1401-Pad1)
- removed copper zone on In2.Cu, net Net-(D1401-Pad1)
- removed copper zone on B.Cu, net Net-(D1501-Pad1)
- removed copper zone on In1.Cu, net Net-(D1501-Pad1)
- removed copper zone on In2.Cu, net Net-(D1501-Pad1)
- removed copper zone on B.Cu, net Net-(D1601-Pad1)
- removed copper zone on In1.Cu, net Net-(D1601-Pad1)
- removed copper zone on In2.Cu, net Net-(D1601-Pad1)
- removed copper zone on B.Cu, net Net-(D1701-Pad1)
- removed copper zone on In1.Cu, net Net-(D1701-Pad1)
- removed copper zone on In2.Cu, net Net-(D1701-Pad1)
- removed copper zone on B.Cu, net Net-(D601-Pad1)
- removed copper zone on In1.Cu, net Net-(D601-Pad1)
- removed copper zone on In2.Cu, net Net-(D601-Pad1)
- removed copper zone on B.Cu, net Net-(D701-Pad1)
- removed copper zone on In1.Cu, net Net-(D701-Pad1)
- removed copper zone on In2.Cu, net Net-(D701-Pad1)
- removed copper zone on B.Cu, net Net-(D801-Pad1)
- removed copper zone on In1.Cu, net Net-(D801-Pad1)
- removed copper zone on In2.Cu, net Net-(D801-Pad1)
- removed copper zone on B.Cu, net Net-(D901-Pad1)
- removed copper zone on In1.Cu, net Net-(D901-Pad1)
- removed copper zone on In2.Cu, net Net-(D901-Pad1)
Other:
- board size 306.9 x 44.7 mm -> 200 x 50 mm
