File: OmniAnt/OmniAnt.kicad_pcb (KiCad board)
At the start: 4 copper layers, 200 x 50 mm, 228 parts, among them J101 USB_B_Micro, J102 Conn_01x02_Pin, J103 Conn_01x04_Pin, J104 Conn_01x02_Pin, J105 Conn_01x02_Pin, J106 XT30PW-M, J107 XT30PW-M, J108 XT30PW-M, J109 XT30PW-M, J110 Conn_01x01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

Commit message: Last Commit At eMatrix.
Parts:
- moved R304 0.85 mm to (185.4, 91.5)
Routing:
- net GND: track 8.12 -> 9.45 mm
- net Net-(U301-FG): track 1.45 -> 2.30 mm
